File: Thermo_Sheild_TwylaBorck/Uno_Shield_ThermoPro.kicad_pcb (KiCad board)
At the start: 2 copper layers, 68.6 x 53.3 mm, 20 parts, among them J1 Power, J2 Digital/PWM, J3 Analog, J4 Digital/PWM, J5 CONN_GYRO, J6 CONN_DISPLAY, J7 CONN_TEMP, SW1 SW_SPST, SW2 SW_SPST, SW3 SW_SPST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

Commit message: added name to silkscreen
Other:
- board text added: "Twyla Borck V 1.0 02/04/25"
Changed lines of the file:
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@@
+		)
+	)
+	(gr_text "Twyla Borck\nV 1.0\n02/04/25"
+		(at 100.5 51.5 0)
+		(layer "F.SilkS")
+		(effects
+			(font
+				(size 1 1)
+				(thickness 0.15)
+			)
+			(justify left bottom)
 		)
 	)
